Commit message: Add urdf for the fridge

File: urdf/dm_shelves.urdf (robot description, URDF)
Before this commit: robot dm_shelves, 79 links, 78 joints
Links:
- removed link room_link
- removed link shelf_1_level_1_divider_10_link
- removed link shelf_1_level_1_divider_1_link
- removed link shelf_1_level_1_divider_2_link
- removed link shelf_1_level_1_divider_3_link
- removed link shelf_1_level_1_divider_4_link
- removed link shelf_1_level_1_divider_5_link
- removed link shelf_1_level_1_divider_6_link
- removed link shelf_1_level_1_divider_7_link
- removed link shelf_1_level_1_divider_8_link
- removed link shelf_1_level_1_divider_9_link
- removed link shelf_1_level_2_divider_10_link
- removed link shelf_1_level_2_divider_1_link
- removed link shelf_1_level_2_divider_2_link
- removed link shelf_1_level_2_divider_3_link
- removed link shelf_1_level_2_divider_4_link
- removed link shelf_1_level_2_divider_5_link
- removed link shelf_1_level_2_divider_6_link
- removed link shelf_1_level_2_divider_7_link
- removed link shelf_1_level_2_divider_8_link
- removed link shelf_1_level_2_divider_9_link
- removed link shelf_1_level_2_left_support_link
- removed link shelf_1_level_2_link
- removed link shelf_1_level_2_right_support_link
- removed link shelf_1_level_3_divider_10_link
- removed link shelf_1_level_3_divider_1_link
- removed link shelf_1_level_3_divider_2_link
- removed link shelf_1_level_3_divider_3_link
- removed link shelf_1_level_3_divider_4_link
- removed link shelf_1_level_3_divider_5_link
- removed link shelf_1_level_3_divider_6_link
- removed link shelf_1_level_3_divider_7_link
- removed link shelf_1_level_3_divider_8_link
- removed link shelf_1_level_3_divider_9_link
- removed link shelf_1_level_3_left_support_link
- removed link shelf_1_level_3_link
- removed link shelf_1_level_3_right_support_link
- removed link shelf_1_level_4_divider_10_link
- removed link shelf_1_level_4_divider_1_link
- removed link shelf_1_level_4_divider_2_link
- removed link shelf_1_level_4_divider_3_link
- removed link shelf_1_level_4_divider_4_link
- removed link shelf_1_level_4_divider_5_link
- removed link shelf_1_level_4_divider_6_link
- removed link shelf_1_level_4_divider_7_link
- removed link shelf_1_level_4_divider_8_link
- removed link shelf_1_level_4_divider_9_link
- removed link shelf_1_level_4_left_support_link
- removed link shelf_1_level_4_link
- removed link shelf_1_level_4_right_support_link
- removed link shelf_1_level_5_divider_10_link
- removed link shelf_1_level_5_divider_1_link
- removed link shelf_1_level_5_divider_2_link
- removed link shelf_1_level_5_divider_3_link
- removed link shelf_1_level_5_divider_4_link
- removed link shelf_1_level_5_divider_5_link
- removed link shelf_1_level_5_divider_6_link
- removed link shelf_1_level_5_divider_7_link
- removed link shelf_1_level_5_divider_8_link
- removed link shelf_1_level_5_divider_9_link
- removed link shelf_1_level_5_left_support_link
- removed link shelf_1_level_5_link
- removed link shelf_1_level_5_right_support_link
- removed link shelf_2_back
- removed link shelf_2_base
- removed link shelf_2_left_side
- removed link shelf_2_level_0_link
- removed link shelf_2_right_side
- removed link shelf_2_shelf_2_level_1_link
- removed link shelf_2_shelf_2_level_2_link
- removed link shelf_2_shelf_2_level_3_link
- removed link shelf_2_shelf_2_level_4_link
- removed link shelf_2_shelf_2_level_5_link
- added link base_link
- link shelf_1_back: geometry collision box size=0.6 0.12 1; visual box size=0.6 0.12 1
- link shelf_1_base: geometry collision box size=0.6 0.4 0.15; visual box size=0.6 0.4 0.15
- link shelf_1_level_0_link: geometry collision box size=0.48 0.35 0.043; visual box size=0.48 0.35 0.043
- link shelf_1_level_1_left_support_link: geometry collision box size=0.004 0.35 0.12; visual box size=0.004 0.35 0.12
- link shelf_1_level_1_link: geometry collision box size=0.480 0.35 0.043; visual box size=0.480 0.35 0.043
- link shelf_1_level_1_right_support_link: geometry collision box size=0.004 0.35 0.12; visual box size=0.004 0.35 0.12
Joints:
- removed joint shelf_1_level_1_divider_10_joint
- removed joint shelf_1_level_1_divider_1_joint
- removed joint shelf_1_level_1_divider_2_joint
- removed joint shelf_1_level_1_divider_3_joint
- removed joint shelf_1_level_1_divider_4_joint
- removed joint shelf_1_level_1_divider_5_joint
- removed joint shelf_1_level_1_divider_6_joint
- removed joint shelf_1_level_1_divider_7_joint
- removed joint shelf_1_level_1_divider_8_joint
- removed joint shelf_1_level_1_divider_9_joint
- removed joint shelf_1_level_2_divider_10_joint
- removed joint shelf_1_level_2_divider_1_joint
- removed joint shelf_1_level_2_divider_2_joint
- removed joint shelf_1_level_2_divider_3_joint
- removed joint shelf_1_level_2_divider_4_joint
- removed joint shelf_1_level_2_divider_5_joint
- removed joint shelf_1_level_2_divider_6_joint
- removed joint shelf_1_level_2_divider_7_joint
- removed joint shelf_1_level_2_divider_8_joint
- removed joint shelf_1_level_2_divider_9_joint
- removed joint shelf_1_level_2_joint
- removed joint shelf_1_level_2_left_support_joint
- removed joint shelf_1_level_2_right_support_joint
- removed joint shelf_1_level_3_divider_10_joint
- removed joint shelf_1_level_3_divider_1_joint
- removed joint shelf_1_level_3_divider_2_joint
- removed joint shelf_1_level_3_divider_3_joint
- removed joint shelf_1_level_3_divider_4_joint
- removed joint shelf_1_level_3_divider_5_joint
- removed joint shelf_1_level_3_divider_6_joint
- removed joint shelf_1_level_3_divider_7_joint
- removed joint shelf_1_level_3_divider_8_joint
- removed joint shelf_1_level_3_divider_9_joint
- removed joint shelf_1_level_3_joint
- removed joint shelf_1_level_3_left_support_joint
- removed joint shelf_1_level_3_right_support_joint
- removed joint shelf_1_level_4_divider_10_joint
- removed joint shelf_1_level_4_divider_1_joint
- removed joint shelf_1_level_4_divider_2_joint
- removed joint shelf_1_level_4_divider_3_joint
- removed joint shelf_1_level_4_divider_4_joint
- removed joint shelf_1_level_4_divider_5_joint
- removed joint shelf_1_level_4_divider_6_joint
- removed joint shelf_1_level_4_divider_7_joint
- removed joint shelf_1_level_4_divider_8_joint
- removed joint shelf_1_level_4_divider_9_joint
- removed joint shelf_1_level_4_joint
- removed joint shelf_1_level_4_left_support_joint
- removed joint shelf_1_level_4_right_support_joint
- removed joint shelf_1_level_5_divider_10_joint
- removed joint shelf_1_level_5_divider_1_joint
- removed joint shelf_1_level_5_divider_2_joint
- removed joint shelf_1_level_5_divider_3_joint
- removed joint shelf_1_level_5_divider_4_joint
- removed joint shelf_1_level_5_divider_5_joint
- removed joint shelf_1_level_5_divider_6_joint
- removed joint shelf_1_level_5_divider_7_joint
- removed joint shelf_1_level_5_divider_8_joint
- removed joint shelf_1_level_5_divider_9_joint
- removed joint shelf_1_level_5_joint
- removed joint shelf_1_level_5_left_support_joint
- removed joint shelf_1_level_5_right_support_joint
- removed joint shelf_2_base_back_joint
- removed joint shelf_2_base_left_joint
- removed joint shelf_2_base_right_joint
- removed joint shelf_2_joint
- removed joint shelf_2_level_0_joint
- removed joint shelf_2_shelf_2_level_1_joint
- removed joint shelf_2_shelf_2_level_2_joint
- removed joint shelf_2_shelf_2_level_3_joint
- removed joint shelf_2_shelf_2_level_4_joint
- removed joint shelf_2_shelf_2_level_5_joint
- joint shelf_1_base_back_joint: origin xyz=0 0.365 1 -> xyz=0 0.2 0.55
- joint shelf_1_joint: origin xyz=4.3223 -0.2415761 0.08515 rpy=0 0 -1.5756 -> xyz=0.0 -0.2415761 0.08515 rpy=0 0 -1.5756; parent room_link -> base_link
- joint shelf_1_level_1_left_support_joint: origin xyz=-0.494 0 -0.06 -> xyz=-0.24 0 -0.06
- joint shelf_1_level_1_right_support_joint: origin xyz=0.494 0 -0.06 -> xyz=0.24 0 -0.06
